File: hwrxsnes/rx.sch (KiCad schematic (older format))
At the start: 20 parts, among them IC1 ATMEGA328-A, P1 +5v, P2 Clock, P3 Latch, P4 Data, P5 GND, P6 nRF, P7 ISP, P8 RX, P9 TX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

Commit message: v2
* Schematic revs:
  * TVS protection on TX
  * TX voltage divider moved after the power switch
  * RX adds crystal to run at 16MHz
RX software tested w/ a real console.
Parts:
- added C6, C7: 22p, SMD_Packages:SMD-0402_c, symbol C
- added X1: CRYSTAL, nesRF:TSX-3225, symbol CRYSTAL
- P8, P9: footprint (none) -> nesRF:Small_1x_Pad
Connections:
- net +5V: now also C4.2
- net Data: now also IC1.26 ((PCINT11/ADC3)PC3); no longer IC1.2 ((PCINT20/XCK/T0)PD4)
- net GND: now also C6.1, C7.1; no longer C4.1
- net Green: now also IC1.24 ((PCINT9/ADC1)PC1); no longer IC1.25 ((PCINT10/ADC2)PC2)
- net Yellow: now also IC1.25 ((PCINT10/ADC2)PC2); no longer IC1.24 ((PCINT9/ADC1)PC1)
- net ~RST: now also C4.1; no longer C4.2
- net XTAL1: now reaches IC1.7 ((PCINT6/XTAL1/TOSC1)PB6)
- net XTAL1: now also C6.2, X1.2
- net XTAL2: now reaches IC1.8 ((PCINT7/XTAL2/TOSC2)PB7)
- net XTAL2: now also C7.2, X1.1
- no-connect marks 12 -> 10
Other:
- moved on the sheet: C1, C2, C3, C4, C5, D1, IC1, P1, P2, P3, P4, P5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

Commit message: end-to-end working on breadboard
Parts:
- removed C6, C7: 22p, SMD_Packages:SMD-0402_c, symbol C
- removed X1: CRYSTAL, nesRF:TSX-3225, symbol CRYSTAL
- C2: value 1u -> 0.1u
- R3: value 120 -> 180
Connections:
- net XTAL1: no longer names the net of IC1.7 ((PCINT6/XTAL1/TOSC1)PB6)
- net XTAL2: no longer names the net of IC1.8 ((PCINT7/XTAL2/TOSC2)PB7)
- no-connect marks 10 -> 12
Changed lines of the file:
@@
 Sheet 1 1
 Title "nesRF Receiver (SNES)"
-Date "Sunday, January 04, 2015"
-Rev "v2"
+Date "Monday, January 26, 2015"
+Rev "v3"
 Comp ""
 Comment1 ""
@@
 P 1100 900
 F 0 "C2" H 1100 1000 40  0000 L CNN
-F 1 "1u" H 1106 815 40  0000 L CNN
+F 1 "0.1u" H 1106 815 40  0000 L CNN
 F 2 "SMD_Packages:SMD-0402_c" H 1138 750 30  0001 C CNN
 F 3 "" H 1100 900 60  0000 C CNN
@@
 P 5750 2800
 F 0 "R3" V 5830 2800 40  0000 C CNN
-F 1 "120" V 5757 2801 40  0000 C CNN
+F 1 "180" V 5757 2801 40  0000 C CNN
 F 2 "SMD_Packages:SMD-0402_r" V 5680 2800 30  0001 C CNN
 F 3 "" H 5750 2800 30  0000 C CNN
@@
 	1    0    0    -1
 $EndComp
-$Comp
-L CRYSTAL X1
-U 1 1 54A98B41
-P 5300 2200
-F 0 "X1" H 5300 2350 60  0000 C CNN
-F 1 "CRYSTAL" H 5300 2050 60  0000 C CNN
-F 2 "nesRF:TSX-3225" H 5300 2200 60  0001 C CNN
-F 3 "" H 5300 2200 60  0000 C CNN
-	1    5300 2200
-	0    -1   -1   0
-$EndComp
 Wire Wire Line
 	6900 850  6900 800
 Wire Wire Line
 	6850 850  6900 850
-Wire Wire Line
-	6100 2500 6100 2850
 Wire Wire Line
 	6000 2800 6100 2800
@@
 Connection ~ 1850 1800
 Wire Wire Line
-	1850 2500 1850 1800
+	1850 1800 1850 2500
 Wire Wire Line
 	2000 1800 2000 2100
@@
 Connection ~ 2700 750
 Connection ~ 1250 3450
-Wire Wire Line
-	3900 2500 5300 2500
-Wire Wire Line
-	3900 2400 5050 2400
-Wire Wire Line
-	5050 1900 5300 1900
-$Comp
-L C C7
-U 1 1 54A98DBE
-P 5500 2500
-F 0 "C7" H 5500 2600 40  0000 L CNN
-F 1 "22p" H 5506 2415 40  0000 L CNN
-F 2 "SMD_Packages:SMD-0402_c" H 5538 2350 30  0001 C CNN
-F 3 "" H 5500 2500 60  0000 C CNN
-	1    5500 2500
-	0    1    1    0
-$EndComp
-Wire Wire Line
-	5050 2400 5050 1900
-$Comp
-L C C6
-U 1 1 54A99077
-P 5500 1900
-F 0 "C6" H 5500 2000 40  0000 L CNN
-F 1 "22p" H 5506 1815 40  0000 L CNN
-F 2 "SMD_Packages:SMD-0402_c" H 5538 1750 30  0001 C CNN
-F 3 "" H 5500 1900 60  0000 C CNN
-	1    5500 1900
-	0    1    1    0
-$EndComp
-Wire Wire Line
-	5700 1900 5700 2500
-Wire Wire Line
-	5700 2500 6100 2500
 Connection ~ 6100 2800
 Wire Wire Line
@@
 Wire Wire Line
 	1550 1750 1550 1800
-Text Label 4650 2400 0    60   ~ 0
-XTAL1
-Text Label 4650 2500 0    60   ~ 0
-XTAL2
 NoConn ~ 3900 3800
 Text Label 2700 750  0    60   ~ 0
 2.5v
+Wire Wire Line
+	6100 2800 6100 2850
+NoConn ~ 3900 2400
+NoConn ~ 3900 2500
 $EndSCHEMATC
