File: hwrxnes/rx-nessat.kicad_pcb (KiCad board)
At the start: 2 copper layers, 60.2 x 38.1 mm, 20 parts, among them IC1 ATMEGA328-A, P1 PORT1, P2 PORT2, P3 ISP, P4 nRF, P5 RX, P6 TX, U1 TCR2EF, X1 CRYSTAL

Commit message: routing tweaks
Parts:
- moved R1 13.0 mm to (32.8, 47.8), turned to 180 degrees
- moved C2 10.3 mm to (32.8, 49.8), turned to 180 degrees
- moved U1 6.60 mm to (62.3, 33.5)
- moved C1 2.71 mm to (65.0, 34.0)
- moved R3 0.51 mm to (76.5, 47.0)
- moved C3 0.36 mm to (46.0, 53.8)
Connections:
- IC1 pad 2: Net-(IC1-Pad2) -> /D4_2
- IC1 pad 25: /D4_2 -> Net-(IC1-Pad25)
Routing:
- net /D3_2: track 44.1 -> 20.7 mm, vias 2 -> 0
- net +5V: track 145.5 -> 130.9 mm, vias 1 -> 0
- net GND: track 86.4 -> 99.5 mm
- net /D4_2: track 18.2 -> 8.32 mm
- net /~RST: track 39.5 -> 32.7 mm
- net /2.5v: track 14.6 -> 10.9 mm
- net /LATCH2: track 17.8 -> 19.3 mm
- net /D0_2: track 26.4 -> 25.4 mm
- net /LEDCommon: track 4.38 -> 3.87 mm
- net /CLK2: vias 0 -> 1
