File: hwrxnes/rx-nessat.sch (KiCad schematic (older format))
At the start: 20 parts, among them IC1 ATMEGA328-A, P1 PORT1, P2 PORT2, P3 ISP, P4 nRF, P5 RX, P6 TX, U1 TCR2EF, X1 CRYSTAL

Commit message: routing tweaks
Connections:
- net D4_2: now also IC1.2 ((PCINT20/XCK/T0)PD4); no longer IC1.25 ((PCINT10/ADC2)PC2)
Changed lines of the file:
@@
 LIBS:valves
 LIBS:nesrf
-LIBS:rx-cache
+LIBS:rx-nessat-cache
 EELAYER 25 0
 EELAYER END
@@
 Text Label 4250 2500 0    60   ~ 0
 XTAL2
-NoConn ~ 3900 3800
 Wire Wire Line
 	6250 1500 6250 2500
@@
 Text Label 3900 2750 0    60   ~ 0
 D3_2
-Text Label 3900 2850 0    60   ~ 0
+Text Label 3900 3800 0    60   ~ 0
 D4_2
+NoConn ~ 3900 2850
 $EndSCHEMATC
